File: 1.54in display/hardware/1.54in.sch (EAGLE design)
At the start: 41 parts, among them J2 MICRO-SD_CARD_SOCKETPUSH-PUSH, Q1 310mA/60V/1.6Ω, U2 3.3V, U4 23K640

Commit message: documentation
Parts:
- added LOGO1: OSHW-LOGOS, SparkFun-Aesthetics:OSHW-LOGOS
Other:
- note added: "5V or 3.3V depending on logic level"
- note added: "Ciara Jekel"
- note added: "Connector"
- note added: "Level Shifting"
- note added: "SPI Pull-Ups"
- note removed: "SPI"
- moved on the sheet: C14, C15, C16, J1, R3, R5, R6, U$3, U2, U4

Commit message: minor rev
Parts:
- R2: value 0.47ohm || 3ohm -> 0.47ohm
Changed lines of the file:
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@@
 <part name="SUPPLY5" library="SparkFun-PowerSymbols" deviceset="3.3V" device=""/>
 <part name="R1" library="SparkFun-Resistors" deviceset="10KOHM" device="-0603-1/10W-1%" value="10k"/>
-<part name="R2" library="SparkFun-Resistors" deviceset="RESISTOR" device="0603" value="0.47ohm || 3ohm"/>
+<part name="R2" library="SparkFun-Resistors" deviceset="RESISTOR" device="0603" value="0.47ohm"/>
 <part name="GND13" library="SparkFun-PowerSymbols" deviceset="GND" device=""/>
 <part name="GND14" library="SparkFun-PowerSymbols" deviceset="GND" device=""/>
