File: 1.54in display/hardware/Production/1.54in-Panel.brd (EAGLE design)
At the start: 109.5 x 96.8 mm, 275 parts, among them J2 MICRO-SD_CARD_SOCKETPUSH-PUSH, J4 MICRO-SD_CARD_SOCKETPUSH-PUSH, J6 MICRO-SD_CARD_SOCKETPUSH-PUSH, J8 MICRO-SD_CARD_SOCKETPUSH-PUSH, Q1 310mA/60V/1.6Ω, Q2 310mA/60V/1.6Ω, Q3 310mA/60V/1.6Ω, Q4 310mA/60V/1.6Ω, U1 3.3V, U2 3.3V, U3 23K640, U4 23K640, U5 3.3V, U6 23K640, U7 3.3V, U8 23K640

Commit message: minor rev
Parts:
- removed U$117: (no value), buzzard_labels (33):D##C9
- removed U$118: (no value), buzzard_labels (33):GND11
- removed U$119: (no value), buzzard_labels (33):5V10
- removed U$120: (no value), buzzard_labels (33):3SPI0
- added LOGO1, LOGO2, LOGO3, LOGO4: OSHW-LOGOS, SparkFun-Aesthetics:OSHW-LOGO-S
- R14, R2, R20, R8: value 0.47ohm || 3ohm -> 0.47ohm
- U$100: value (none) -> SPARKX-LOGO4; device buzzard_labels (24):SR#CS1 -> SparkX:SPARKX-MEDIUM
- U$101: device buzzard_labels (25):MISO1 -> buzzard_labels (30):3_COLOR2
- U$102: device buzzard_labels (25):MOSI0 -> buzzard_labels (30):1#54#1
- U$103: device buzzard_labels (25):SCK2 -> buzzard_labels (32):#BUSY1
- U$104: device buzzard_labels (27):#BUSY0 -> buzzard_labels (32):#RST2
- U$105: value SPARKX-LOGO4 -> (none); device SparkX:SPARKX-MEDIUM -> buzzard_labels (32):MISO3
- U$106: device buzzard_labels (29):EINK_DISPLAY0 -> buzzard_labels (32):MOSI4
- U$107: device buzzard_labels (30):3_COLOR2 -> buzzard_labels (32):SCK5
- U$108: device buzzard_labels (30):1#54#1 -> buzzard_labels (32):SD#CS6
- U$109: device buzzard_labels (32):#BUSY1 -> buzzard_labels (32):SR#CS7
- U$110: device buzzard_labels (32):#RST2 -> buzzard_labels (32):D#CS8
- U$111: device buzzard_labels (32):MISO3 -> buzzard_labels (33):D##C9
- U$112: device buzzard_labels (32):MOSI4 -> buzzard_labels (33):GND11
- U$113: device buzzard_labels (32):SCK5 -> buzzard_labels (33):3SPI0
- U$114: device buzzard_labels (32):SD#CS6 -> buzzard_power:VCC1
- U$115, U$85: device buzzard_labels (32):SR#CS7 -> buzzard_power:VCC1
- U$116: device buzzard_labels (32):D#CS8 -> buzzard_labels (35):EPAPER_DISPLAY5
- U$13: device buzzard_labels (22):5V8 -> buzzard_power:VCC1
- U$18: value (none) -> 24_PIN_FPC_0.5MM; device buzzard_labels (29):EINK_DISPLAY0 -> ePaper:24_PIN_FPC_0.5MM
- U$2: device SparkFun-Aesthetics:OSHW-LOGO-S -> buzzard_power:VCC1
- U$21: value 24_PIN_FPC_0.5MM -> (none); device ePaper:24_PIN_FPC_0.5MM -> buzzard_labels (35):EPAPER_DISPLAY5
- U$22: value (none) -> TXB0108DQSR; device SparkFun-Aesthetics:OSHW-LOGO-S -> SparkFun-IC-Comms:UFDFN-20
- U$32: device buzzard_labels (33):5V10 -> buzzard_labels (22):D##C10
- U$33: value TXB0108DQSR -> (none); device SparkFun-IC-Comms:UFDFN-20 -> buzzard_labels (22):#RST1
- U$34: device buzzard_labels (22):D##C10 -> buzzard_labels (22):GND9
- U$35: device buzzard_labels (22):#RST1 -> buzzard_labels (23):D#CS2
- U$36: device buzzard_labels (22):5V8 -> buzzard_labels (23):SD#CS0
- U$37: device buzzard_labels (22):GND9 -> buzzard_labels (24):SR#CS1
- U$38: device buzzard_labels (23):D#CS2 -> buzzard_labels (25):MISO1
- U$39: device buzzard_labels (23):SD#CS0 -> buzzard_labels (25):MOSI0
- U$40: device buzzard_labels (24):SR#CS1 -> buzzard_labels (25):SCK2
- U$41: device buzzard_labels (25):MISO1 -> buzzard_labels (27):#BUSY0
- U$42: value (none) -> SPARKX-LOGO4; device buzzard_labels (25):MOSI0 -> SparkX:SPARKX-MEDIUM
- U$43: device buzzard_labels (25):SCK2 -> buzzard_labels (30):3_COLOR2
- U$44: device buzzard_labels (27):#BUSY0 -> buzzard_labels (30):1#54#1
- U$45: value SPARKX-LOGO4 -> (none); device SparkX:SPARKX-MEDIUM -> buzzard_labels (32):#BUSY1
- U$46: device buzzard_labels (29):EINK_DISPLAY0 -> buzzard_labels (32):#RST2
- U$47: device buzzard_labels (30):3_COLOR2 -> buzzard_labels (32):MISO3
- U$48: device buzzard_labels (30):1#54#1 -> buzzard_labels (32):MOSI4
- U$49: device buzzard_labels (32):#BUSY1 -> buzzard_labels (32):SCK5
- U$50: device buzzard_labels (32):#RST2 -> buzzard_labels (32):SD#CS6
- U$51: device buzzard_labels (32):MISO3 -> buzzard_labels (32):SR#CS7
- U$52: device buzzard_labels (32):MOSI4 -> buzzard_labels (32):D#CS8
- U$53: device buzzard_labels (32):SCK5 -> buzzard_labels (33):D##C9
- U$54: device buzzard_labels (32):SD#CS6 -> buzzard_labels (33):GND11
- U$55: device buzzard_labels (32):SR#CS7 -> buzzard_labels (33):3SPI0
- U$56, U$86: device buzzard_labels (32):D#CS8 -> buzzard_power:VCC1
- U$57: device buzzard_labels (33):D##C9 -> buzzard_power:VCC1
- U$58: device buzzard_labels (33):GND11 -> buzzard_labels (35):EPAPER_DISPLAY5
- U$59: value (none) -> 24_PIN_FPC_0.5MM; device buzzard_labels (33):5V10 -> ePaper:24_PIN_FPC_0.5MM
- U$60: value (none) -> TXB0108DQSR; device buzzard_labels (33):3SPI0 -> SparkFun-IC-Comms:UFDFN-20
- U$61: value 24_PIN_FPC_0.5MM -> (none); device ePaper:24_PIN_FPC_0.5MM -> buzzard_labels (22):D##C10
- U$62: device SparkFun-Aesthetics:OSHW-LOGO-S -> buzzard_labels (22):#RST1
- U$63: value TXB0108DQSR -> (none); device SparkFun-IC-Comms:UFDFN-20 -> buzzard_labels (22):GND9
- U$64: device buzzard_labels (22):D##C10 -> buzzard_labels (23):D#CS2
- U$65: device buzzard_labels (22):#RST1 -> buzzard_labels (23):SD#CS0
- U$66: device buzzard_labels (22):5V8 -> buzzard_labels (24):SR#CS1
- U$67: device buzzard_labels (22):GND9 -> buzzard_labels (25):MISO1
- U$68: device buzzard_labels (23):D#CS2 -> buzzard_labels (25):MOSI0
- U$69: device buzzard_labels (23):SD#CS0 -> buzzard_labels (25):SCK2
- U$70: device buzzard_labels (24):SR#CS1 -> buzzard_labels (27):#BUSY0
- U$71: value (none) -> SPARKX-LOGO4; device buzzard_labels (25):MISO1 -> SparkX:SPARKX-MEDIUM
- U$72: device buzzard_labels (25):MOSI0 -> buzzard_labels (30):3_COLOR2
- U$73: device buzzard_labels (25):SCK2 -> buzzard_labels (30):1#54#1
- U$74: device buzzard_labels (27):#BUSY0 -> buzzard_labels (32):#BUSY1
- U$75: value SPARKX-LOGO4 -> (none); device SparkX:SPARKX-MEDIUM -> buzzard_labels (32):#RST2
- U$76: device buzzard_labels (29):EINK_DISPLAY0 -> buzzard_labels (32):MISO3
- U$77: device buzzard_labels (30):3_COLOR2 -> buzzard_labels (32):MOSI4
- U$78: device buzzard_labels (30):1#54#1 -> buzzard_labels (32):SCK5
- U$79: device buzzard_labels (32):#BUSY1 -> buzzard_labels (32):SD#CS6
- U$80: device buzzard_labels (32):#RST2 -> buzzard_labels (32):SR#CS7
- U$81: device buzzard_labels (32):MISO3 -> buzzard_labels (32):D#CS8
- U$82: device buzzard_labels (32):MOSI4 -> buzzard_labels (33):D##C9
- U$83: device buzzard_labels (32):SCK5 -> buzzard_labels (33):GND11
- U$84: device buzzard_labels (32):SD#CS6 -> buzzard_labels (33):3SPI0
- U$87: device buzzard_labels (33):D##C9 -> buzzard_labels (35):EPAPER_DISPLAY5
- U$88: value (none) -> 24_PIN_FPC_0.5MM; device buzzard_labels (33):GND11 -> ePaper:24_PIN_FPC_0.5MM
- U$89: value (none) -> TXB0108DQSR; device buzzard_labels (33):5V10 -> SparkFun-IC-Comms:UFDFN-20
- U$90: device buzzard_labels (33):3SPI0 -> buzzard_labels (22):D##C10
- U$91: value 24_PIN_FPC_0.5MM -> (none); device ePaper:24_PIN_FPC_0.5MM -> buzzard_labels (22):#RST1
- U$92: device SparkFun-Aesthetics:OSHW-LOGO-S -> buzzard_labels (22):GND9
- U$93: value TXB0108DQSR -> (none); device SparkFun-IC-Comms:UFDFN-20 -> buzzard_labels (23):D#CS2
- U$94: device buzzard_labels (22):D##C10 -> buzzard_labels (23):SD#CS0
- U$95: device buzzard_labels (22):#RST1 -> buzzard_labels (24):SR#CS1
- U$96: device buzzard_labels (22):5V8 -> buzzard_labels (25):MISO1
- U$97: device buzzard_labels (22):GND9 -> buzzard_labels (25):MOSI0
- U$98: device buzzard_labels (23):D#CS2 -> buzzard_labels (25):SCK2
- U$99: device buzzard_labels (23):SD#CS0 -> buzzard_labels (27):#BUSY0
- U3, U4, U6, U8: device SparkFun-IC-Memory:SOIC-8 -> SparkFun-IC-Memory:SO08
- moved U$60 84.0 mm to (8.76, 56.1), turned to 90 degrees
- moved U$88 73.6 mm to (79.2, 57.5), flipped to the top, turned to 90 degrees
- moved U$21 55.0 mm to (25.7, 31.5), turned to 0 degrees
- moved U$59 53.6 mm to (34.3, 57.5), flipped to the top, turned to 90 degrees
- moved U$18 50.8 mm to (79.2, 18.9), turned to 90 degrees
- moved U$89 49.7 mm to (53.7, 56.1), flipped to the top, turned to 90 degrees
- moved U$62 47.5 mm to (1.40, 67.8)
- moved U$32 41.3 mm to (46.4, 11.4), flipped to the top
- moved U$92 40.2 mm to (46.5, 47.5)
- moved U$2 40.1 mm to (1.40, 6.35)
- moved U$100 37.2 mm to (78.4, 74.2)
- moved U$22 35.5 mm to (53.7, 17.5), turned to 90 degrees
- moved U$91 34.5 mm to (46.4, 67.8), turned to 0 degrees
- moved U$42 33.9 mm to (78.4, 35.6)
- moved U$61 33.7 mm to (1.40, 50.0), turned to 0 degrees
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Connections:
- net !BUSY1: now also U$18.9; no longer U$21.9
- net !BUSY2: now also U$59.9; no longer U$61.9
- net !BUSY3: now also U$88.9; no longer U$91.9
- net !CS!(D)1: now also U$18.12, U$22.2; no longer U$21.12, U$33.2
- net !CS!(D)2: now also U$59.12, U$60.2; no longer U$61.12, U$63.2
- net !CS!(D)3: now also U$88.12, U$89.2; no longer U$91.12, U$93.2
- net !CS!(SD)1: now also U$22.4; no longer U$33.4
- net !CS!(SD)2: now also U$60.4; no longer U$63.4
- net !CS!(SD)3: now also U$89.4; no longer U$93.4
- net !CS!(SR)1: now also U$22.3; no longer U$33.3
- net !CS!(SR)2: now also U$60.3; no longer U$63.3
- net !CS!(SR)3: now also U$89.3; no longer U$93.3
- net !RES1: now also U$18.10, U$22.10; no longer U$21.10, U$33.10
- net !RES2: now also U$59.10, U$60.10; no longer U$61.10, U$63.10
- net !RES3: now also U$88.10, U$89.10; no longer U$91.10, U$93.10
- net 3.3V1: now also U$18.15, U$18.16, U$22.5, U$22.6; no longer U$21.15, U$21.16, U$33.5, U$33.6
- net 3.3V2: now also U$59.15, U$59.16, U$60.5, U$60.6; no longer U$61.15, U$61.16, U$63.5, U$63.6
- net 3.3V3: now also U$88.15, U$88.16, U$89.5, U$89.6; no longer U$91.15, U$91.16, U$93.5, U$93.6
- net 5V1: now also U$22.16; no longer U$33.16
- net 5V2: now also U$60.16; no longer U$63.16
- net 5V3: now also U$89.16; no longer U$93.16
- net 5V_!CS!(D)1: now also U$22.19; no longer U$33.19
- net 5V_!CS!(D)2: now also U$60.19; no longer U$63.19
- net 5V_!CS!(D)3: now also U$89.19; no longer U$93.19
- net 5V_!CS!(SD)1: now also U$22.17; no longer U$33.17
- net 5V_!CS!(SD)2: now also U$60.17; no longer U$63.17
- net 5V_!CS!(SD)3: now also U$89.17; no longer U$93.17
- net 5V_!CS!(SR)1: now also U$22.18; no longer U$33.18
- net 5V_!CS!(SR)2: now also U$60.18; no longer U$63.18
- net 5V_!CS!(SR)3: now also U$89.18; no longer U$93.18
- net 5V_!RES1: now also U$22.11; no longer U$33.11
- net 5V_!RES2: now also U$60.11; no longer U$63.11
- net 5V_!RES3: now also U$89.11; no longer U$93.11
- net 5V_D/!C1: now also U$22.20; no longer U$33.20
- net 5V_D/!C2: now also U$60.20; no longer U$63.20
- net 5V_D/!C3: now also U$89.20; no longer U$93.20
- net 5V_MISO1: now also U$22.12; no longer U$33.12
- net 5V_MISO2: now also U$60.12; no longer U$63.12
- net 5V_MISO3: now also U$89.12; no longer U$93.12
- net 5V_MOSI1: now also U$22.13; no longer U$33.13
- net 5V_MOSI2: now also U$60.13; no longer U$63.13
- net 5V_MOSI3: now also U$89.13; no longer U$93.13
- net 5V_SCLK1: now also U$22.14; no longer U$33.14
- net 5V_SCLK2: now also U$60.14; no longer U$63.14
- net 5V_SCLK3: now also U$89.14; no longer U$93.14
- net BS1: now also U$18.8; no longer U$21.8
- net BS2: now also U$59.8; no longer U$61.8
- net BS3: now also U$88.8; no longer U$91.8
- net D/!C1: now also U$18.11, U$22.1; no longer U$21.11, U$33.1
- net D/!C2: now also U$59.11, U$60.1; no longer U$61.11, U$63.1
- net D/!C3: now also U$88.11, U$89.1; no longer U$91.11, U$93.1
- net GDR1: now also U$18.2; no longer U$21.2
- net GDR2: now also U$59.2; no longer U$61.2
- net GDR3: now also U$88.2; no longer U$91.2
- net GND1: now also U$18.17, U$22.15; no longer U$21.17, U$33.15
- net GND2: now also U$59.17, U$60.15; no longer U$61.17, U$63.15
- net GND3: now also U$88.17, U$89.15; no longer U$91.17, U$93.15
- net MISO1: now also U$22.9; no longer U$33.9
- net MISO2: now also U$60.9; no longer U$63.9
- net MISO3: now also U$89.9; no longer U$93.9
- net MOSI1: now also U$18.14, U$22.8; no longer U$21.14, U$33.8
- net MOSI2: now also U$59.14, U$60.8; no longer U$61.14, U$63.8
- net MOSI3: now also U$88.14, U$89.8; no longer U$91.14, U$93.8
- net PREVGH1: now also U$18.21; no longer U$21.21
- net PREVGH2: now also U$59.21; no longer U$61.21
- net PREVGH3: now also U$88.21; no longer U$91.21
- net PREVGL1: now also U$18.23; no longer U$21.23
- net PREVGL2: now also U$59.23; no longer U$61.23
- net PREVGL3: now also U$88.23; no longer U$91.23
- net RESE1: now also U$18.3; no longer U$21.3
- net RESE2: now also U$59.3; no longer U$61.3
- net RESE3: now also U$88.3; no longer U$91.3
- net SCLK1: now also U$18.13, U$22.7; no longer U$21.13, U$33.7
- net SCLK2: now also U$59.13, U$60.7; no longer U$61.13, U$63.7
- net SCLK3: now also U$88.13, U$89.7; no longer U$91.13, U$93.7
- net TSCL1: now also U$18.6; no longer U$21.6
- net TSCL2: now also U$59.6; no longer U$61.6
- net TSCL3: now also U$88.6; no longer U$91.6
- net TSDA1: now also U$18.7; no longer U$21.7
- net TSDA2: now also U$59.7; no longer U$61.7
- net TSDA3: now also U$88.7; no longer U$91.7
- net VCOM1: now also U$18.24; no longer U$21.24
- net VCOM2: now also U$59.24; no longer U$61.24
- net VCOM3: now also U$88.24; no longer U$91.24
- net VDD1: now also U$18.18; no longer U$21.18
- net VDD2: now also U$59.18; no longer U$61.18
- net VDD3: now also U$88.18; no longer U$91.18
- net VGH1: now also U$18.5; no longer U$21.5
- net VGH2: now also U$59.5; no longer U$61.5
- net VGH3: now also U$88.5; no longer U$91.5
- net VGL1: now also U$18.4; no longer U$21.4
- net VGL2: now also U$59.4; no longer U$61.4
- net VGL3: now also U$88.4; no longer U$91.4
- net VPP1: now also U$18.19; no longer U$21.19
- net VPP2: now also U$59.19; no longer U$61.19
- net VPP3: now also U$88.19; no longer U$91.19
- net VSH1: now also U$18.20; no longer U$21.20
- net VSH2: now also U$59.20; no longer U$61.20
- net VSH3: now also U$88.20; no longer U$91.20
- net VSL1: now also U$18.22; no longer U$21.22
- net VSL2: now also U$59.22; no longer U$61.22
- net VSL3: now also U$88.22; no longer U$91.22
Routing:
- net 3.3V3: track 102.5 -> 106.8 mm
- net 3.3V: track 102.5 -> 106.8 mm
- net 3.3V2: track 102.5 -> 106.8 mm
- net 3.3V1: track 102.5 -> 106.8 mm
- net SCLK2: track 52.5 -> 54.1 mm, vias 2 -> 4
- net SCLK: track 52.5 -> 54.1 mm, vias 2 -> 4
- net SCLK1: track 52.5 -> 54.1 mm, vias 2 -> 4
- net SCLK3: track 52.5 -> 54.1 mm, vias 2 -> 4
- net MOSI: track 51.1 -> 52.6 mm
- net MOSI3: track 51.1 -> 52.6 mm
- net MOSI2: track 51.1 -> 52.6 mm
- net MOSI1: track 51.1 -> 52.6 mm
- net !CS!(SD)2: track 16.5 -> 17.7 mm
- net !CS!(SD): track 16.5 -> 17.7 mm
- net !CS!(SD)3: track 16.5 -> 17.7 mm
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