File: 7.5in display/Hardware/7.5in display.sch (EAGLE design)
At the start: 41 parts, among them J2 MICRO-SD_CARD_SOCKETPUSH-PUSH, Q1 310mA/60V/1.6Ω, U2 3.3V, U4 23K640

Commit message: brds
Other:
- note removed: "3.3v?"
- note removed: "diode ratings ??"
Changed lines of the file:
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@@
 <?xml version="1.0" encoding="utf-8"?>
 <!DOCTYPE eagle SYSTEM "eagle.dtd">
-<eagle version="9.0.1">
+<eagle version="9.1.3">
 <drawing>
 <settings>
@@
 <text x="59.182" y="98.552" size="1.27" layer="97" rot="MR0">BUSY - when low, commands should not be issued</text>
 <text x="60.198" y="101.092" size="1.27" layer="97" rot="MR0">BS - Low = 4 line SPI, High= 3 line SPI</text>
-<text x="43.18" y="167.64" size="1.27" layer="97">diode ratings ??</text>
 <text x="55.88" y="85.09" size="1.27" layer="97" rot="MR180">VDDIO</text>
 <text x="54.102" y="81.28" size="1.27" layer="97" rot="MR0">VCI</text>
@@
 <text x="162.56" y="91.44" size="2.54" layer="97">SPI </text>
 <text x="28.956" y="37.592" size="2.54" layer="97">uSD</text>
-<text x="126.492" y="21.082" size="1.778" layer="97">3.3v?</text>
 <text x="2.54" y="81.28" size="1.778" layer="97">Close this jumper
 to use 3-line SPI</text>
