File: 4.2in display/Hardware/4.2in display.sch (EAGLE design)
At the start: 41 parts, among them J2 MICRO-SD_CARD_SOCKETPUSH-PUSH, Q1 310mA/60V/1.6Ω, U2 3.3V, U4 23K640

Commit message: 4.2 schematic update
Other:
- note added: "Ciara Jekel"
Changed lines of the file:
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@@
 <?xml version="1.0" encoding="utf-8"?>
 <!DOCTYPE eagle SYSTEM "eagle.dtd">
-<eagle version="9.0.1">
+<eagle version="9.1.3">
 <drawing>
 <settings>
@@
 <wire x1="96.52" y1="45.72" x2="248.92" y2="45.72" width="0.1524" layer="97" style="longdash"/>
 <text x="106.68" y="35.56" size="2.54" layer="97">SRAM</text>
+<text x="165.1" y="10.16" size="2.54" layer="97">Ciara Jekel</text>
 </plain>
 <instances>
