File: 4.2in display/Hardware/4.2in display.brd (EAGLE design)
At the start: 33 x 38.1 mm, 73 parts, among them J2 MICRO-SD_CARD_SOCKETPUSH-PUSH, Q1 NMOS, U2 3.3V, U4 23K640

Commit message: Revert "Revert "Revert "asm"""
This reverts commit 13aa5e244575f702f785403d246ecc40f8071a55.
Parts:
- D1, D2: value shtkydio -> 0.5A/40V/420mV
- D3: value shtky dio -> 0.5A/40V/420mV
- Q1: value NMOS -> 310mA/60V/1.6Ω

Commit message: Revert "Revert "asm""
This reverts commit b489ea2ff6e59cc2c3bae19cf3fe86e4ee51237d.
Parts:
- D1, D2: value 0.5A/40V/420mV -> shtkydio
- D3: value 0.5A/40V/420mV -> shtky dio
- Q1: value 310mA/60V/1.6Ω -> NMOS
